File: ad9781.kicad_sch (KiCad schematic)
At the start: 20 parts, among them J1201 142-0701-201, J1202 142-0701-201, U1201 AD9781BCPZ

Commit message: fixed differential pair impedance and length matching. Also fixed DRC errors (trace spacing). These are only layout changes, the schematic remains unchanged.
Connections:
- net D_CLKP: now reaches C1202.2, R1201.2, U1201.3 (CLKP)
- net D_CLKN: now reaches C1203.2, R1202.2, U1201.4 (CLKN)
Changed lines of the file:
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@@
+		)
+	)
+	(label "D_CLKP"
+		(at 91.44 80.01 0)
+		(effects
+			(font
+				(size 1.27 1.27)
+			)
+			(justify left bottom)
 		)
 	)
@@
 		(effects
 			(font
+				(size 1.27 1.27)
+			)
+			(justify left bottom)
+		)
+	)
+	(label "D_CLKN"
+		(at 91.44 101.6 0)
+		(effects
+			(font
