File: ad9781.kicad_sch (KiCad schematic)
At the start: 20 parts, among them J1201 142-0701-201, J1202 142-0701-201, U1201 AD9781BCPZ

Commit message: fixed differential pair impedance and length matching. Also fixed DRC errors (trace spacing). These are only layout changes, the schematic remains unchanged.
Connections:
- net D_CLKP: now reaches C1202.2, R1201.2, U1201.3 (CLKP)
- net D_CLKN: now reaches C1203.2, R1202.2, U1201.4 (CLKN)
Changed lines of the file:
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@@
 (kicad_sch
-	(version 20231120)
+	(version 20250114)
 	(generator "eeschema")
-	(generator_version "8.0")
+	(generator_version "9.0")
 	(paper "A4")
 	(junction
@@
 		)
 	)
+	(label "D_CLKP"
+		(at 91.44 80.01 0)
+		(effects
+			(font
+				(size 1.27 1.27)
+			)
+			(justify left bottom)
+		)
+	)
 	(label "D_P_11"
 		(at 151.13 93.98 180)
-		(fields_autoplaced yes)
 		(effects
 			(font
@@
 	(label "D_P_1"
 		(at 201.93 149.86 0)
-		(fields_autoplaced yes)
 		(effects
 			(font
@@
 	(label "D_N_0"
 		(at 201.93 142.24 0)
-		(fields_autoplaced yes)
 		(effects
 			(font
@@
 	(label "D_N_7"
 		(at 151.13 116.84 180)
-		(fields_autoplaced yes)
 		(effects
 			(font
@@
 	(label "D_N_9"
 		(at 151.13 106.68 180)
-		(fields_autoplaced yes)
 		(effects
 			(font
@@
 	(label "D_P_3"
 		(at 151.13 149.86 180)
-		(fields_autoplaced yes)
 		(effects
 			(font
@@
 	(label "DCI_P"
 		(at 151.13 134.62 180)
-		(fields_autoplaced yes)
 		(effects
 			(font
@@
 	(label "DAC_SDIO"
 		(at 201.93 121.92 0)
-		(fields_autoplaced yes)
 		(effects
 			(font
@@
 	(label "D_P_4"
 		(at 151.13 144.78 180)
-		(fields_autoplaced yes)
 		(effects
 			(font
@@
 	(label "{DAC}"
 		(at 121.92 95.25 180)
-		(fields_autoplaced yes)
 		(effects
 			(font
@@
 	(label "D_P_2"
 		(at 201.93 154.94 0)
-		(fields_autoplaced yes)
 		(effects
 			(font
@@
 	(label "D_N_12"
 		(at 151.13 91.44 180)
-		(fields_autoplaced yes)
 		(effects
 			(font
@@
 	(label "DCI_N"
 		(at 151.13 137.16 180)
-		(fields_autoplaced yes)
 		(effects
 			(font
@@
 	(label "D_N_10"
 		(at 151.13 101.6 180)
-		(fields_autoplaced yes)
 		(effects
 			(font
@@
 	(label "DAC_SDO"
 		(at 201.93 124.46 0)
-		(fields_autoplaced yes)
 		(effects
 			(font
@@
 	(label "D_P_8"
 		(at 151.13 109.22 180)
-		(fields_autoplaced yes)
 		(effects
 			(font
@@
 	(label "D_N_11"
 		(at 151.13 96.52 180)
-		(fields_autoplaced yes)
 		(effects
 			(font
@@
 	(label "D_P_0"
 		(at 201.93 144.78 0)
-		(fields_autoplaced yes)
 		(effects
 			(font
@@
 	(label "DAC_CLKN"
 		(at 31.75 101.6 0)
-		(fields_autoplaced yes)
 		(effects
 			(font
@@
 	(label "D_N_3"
 		(at 151.13 152.4 180)
-		(fields_autoplaced yes)
 		(effects
 			(font
@@
 	(label "DAC_CLKP"
 		(at 31.75 80.01 0)
-		(fields_autoplaced yes)
 		(effects
 			(font
@@
 	(label "{DAC}"
 		(at 219.71 143.51 0)
-		(fields_autoplaced yes)
 		(effects
 			(font
@@
 	(label "D_N_8"
 		(at 151.13 111.76 180)
-		(fields_autoplaced yes)
 		(effects
 			(font
@@
 	(label "DCO_N"
 		(at 151.13 127 180)
-		(fields_autoplaced yes)
 		(effects
 			(font
@@
 	(label "D_P_5"
 		(at 151.13 139.7 180)
-		(fields_autoplaced yes)
 		(effects
 			(font
@@
 	(label "DAC_CSB"
 		(at 201.93 116.84 0)
-		(fields_autoplaced yes)
+		(effects
+			(font
+				(size 1.27 1.27)
+			)
+			(justify left bottom)
+		)
+	)
+	(label "D_CLKN"
+		(at 91.44 101.6 0)
 		(effects
 			(font
@@
 	(label "D_N_13"
 		(at 151.13 86.36 180)
-		(fields_autoplaced yes)
 		(effects
 			(font
@@
 	(label "DCO_P"
 		(at 151.13 124.46 180)
-		(fields_autoplaced yes)
 		(effects
 			(font
@@
 	(label "D_P_7"
 		(at 151.13 114.3 180)
-		(fields_autoplaced yes)
 		(effects
 			(font
@@
 	(label "D_N_6"
 		(at 151.13 121.92 180)
-		(fields_autoplaced yes)
 		(effects
 			(font
@@
 	(label "D_N_5"
 		(at 151.13 142.24 180)
-		(fields_autoplaced yes)
 		(effects
 			(font
@@
 	(label "D_P_12"
 		(at 151.13 88.9 180)
-		(fields_autoplaced yes)
 		(effects
 			(font
@@
 	(label "D_P_9"
 		(at 151.13 104.14 180)
-		(fields_autoplaced yes)
 		(effects
 			(font
@@
 	(label "D_P_10"
 		(at 151.13 99.06 180)
-		(fields_autoplaced yes)
 		(effects
 			(font
@@
 	(label "DAC_SCLK"
 		(at 201.93 119.38 0)
-		(fields_autoplaced yes)
 		(effects
 			(font
@@
 	(label "D_P_13"
 		(at 151.13 83.82 180)
-		(fields_autoplaced yes)
 		(effects
 			(font
@@
 	(label "DAC_RESET"
 		(at 201.93 114.3 0)
-		(fields_autoplaced yes)
 		(effects
 			(font
@@
 	(label "D_P_6"
 		(at 151.13 119.38 180)
-		(fields_autoplaced yes)
 		(effects
 			(font
@@
 	(label "D_N_4"
 		(at 151.13 147.32 180)
-		(fields_autoplaced yes)
 		(effects
 			(font
@@
 	(label "D_N_1"
 		(at 201.93 147.32 0)
-		(fields_autoplaced yes)
 		(effects
 			(font
@@
 	(label "D_N_2"
 		(at 201.93 152.4 0)
-		(fields_autoplaced yes)
 		(effects
 			(font
@@
 		(shape input)
 		(at 224.79 115.57 0)
-		(fields_autoplaced yes)
 		(effects
 			(font
@@
 		(shape input)
 		(at 29.21 82.55 180)
-		(fields_autoplaced yes)
 		(effects
 			(font
@@
 		(shape input)
 		(at 36.83 26.67 180)
-		(fields_autoplaced yes)
 		(effects
 			(font
@@
 		(shape input)
 		(at 121.92 111.76 180)
-		(fields_autoplaced yes)
 		(effects
 			(font
@@
 		(shape input)
 		(at 36.83 39.37 180)
-		(fields_autoplaced yes)
 		(effects
 			(font
@@
 		(shape input)
 		(at 36.83 35.56 180)
-		(fields_autoplaced yes)
 		(effects
 			(font
@@
 		(shape input)
 		(at 36.83 31.75 180)
-		(fields_autoplaced yes)
 		(effects
 			(font
@@
 		(at 229.87 72.39)
 		(size 15.24 7.62)
+		(exclude_from_sim no)
+		(in_bom yes)
+		(on_board yes)
+		(dnp no)
 		(fields_autoplaced yes)
 		(stroke
@@
 		(at 229.87 95.25)
 		(size 15.24 7.62)
+		(exclude_from_sim no)
+		(in_bom yes)
+		(on_board yes)
+		(dnp no)
 		(fields_autoplaced yes)
 		(stroke
