File: diff_se.kicad_sch (KiCad schematic)
At the start: 7 parts

Commit message: fixed differential pair impedance and length matching. Also fixed DRC errors (trace spacing). These are only layout changes, the schematic remains unchanged.
Changed lines of the file:
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@@
 (kicad_sch
-	(version 20231120)
+	(version 20250114)
 	(generator "eeschema")
-	(generator_version "8.0")
+	(generator_version "9.0")
 	(paper "A4")
 	(junction
@@
 		(shape input)
 		(at 50.8 85.09 180)
-		(fields_autoplaced yes)
 		(effects
 			(font
@@
 		(shape input)
 		(at 52.07 95.25 180)
-		(fields_autoplaced yes)
 		(effects
 			(font
@@
 		(shape input)
 		(at 52.07 73.66 180)
-		(fields_autoplaced yes)
 		(effects
 			(font
@@
 		(shape input)
 		(at 220.98 83.82 0)
-		(fields_autoplaced yes)
 		(effects
 			(font
@@
 		(shape input)
 		(at 220.98 88.9 0)
-		(fields_autoplaced yes)
-		(effects
-			(font
+		(effects
+			(font
