File: lmk01801.kicad_sch (KiCad schematic)
At the start: 41 parts, among them J1001 142-0701-201, J1002 U.FL-R-SMT(10), J1003 U.FL-R-SMT(10), J1004 142-0701-201, J1005 U.FL-R-SMT(10), T1001 TCM2-43X+, T1002 TCM2-43X+, U1001 TCP-2-33W+, U1002 LMK01801BISQE/NOPB

Commit message: fixed differential pair impedance and length matching. Also fixed DRC errors (trace spacing). These are only layout changes, the schematic remains unchanged.
Connections:
- net CinP: now reaches C1007.1, R1002.1, T1001.4
- net CinN: now reaches C1006.1, R1002.2, T1001.6
- net aux_clk_n renamed aux_clk_N
- net aux_clk_p renamed aux_clk_P
Changed lines of the file:
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@@
 (kicad_sch
-	(version 20231120)
+	(version 20250114)
 	(generator "eeschema")
-	(generator_version "8.0")
+	(generator_version "9.0")
 	(paper "A4")
 	(bus_alias "LMKuWire"
@@
 	(label "LMK2468_plane"
 		(at 252.73 127 0)
-		(fields_autoplaced yes)
 		(effects
 			(font
@@
 	(label "LMK_CLKout3_N"
 		(at 143.51 78.74 180)
-		(fields_autoplaced yes)
 		(effects
 			(font
@@
 	(label "ADC0_CLK-"
 		(at 135.89 66.04 180)
-		(fields_autoplaced yes)
 		(effects
 			(font
@@
 		)
 	)
-	(label "aux_clk_p"
+	(label "aux_clk_P"
 		(at 246.38 93.98 0)
-		(fields_autoplaced yes)
-		(effects
-			(font
-				(size 1.27 1.27)
-			)
-			(justify left bottom)
-		)
-	)
-	(label "aux_clk_p"
+		(effects
+			(font
+				(size 1.27 1.27)
+			)
+			(justify left bottom)
+		)
+	)
+	(label "aux_clk_P"
 		(at 172.72 149.86 180)
-		(fields_autoplaced yes)
 		(effects
 			(font
@@
 	(label "LMK_CLKout4_P"
 		(at 143.51 104.14 180)
-		(fields_autoplaced yes)
 		(effects
 			(font
@@
 	(label "CLKinP"
 		(at 245.11 78.74 0)
-		(fields_autoplaced yes)
 		(effects
 			(font
@@
 	(label "DAC_CLKN"
 		(at 118.11 111.76 0)
-		(fields_autoplaced yes)
 		(effects
 			(font
@@
 	(label "CLKinN"
 		(at 101.6 151.13 0)
-		(fields_autoplaced yes)
 		(effects
 			(font
@@
 	(label "LMK2468_plane"
 		(at 83.82 33.02 0)
-		(fields_autoplaced yes)
+		(effects
+			(font
+				(size 1.27 1.27)
+			)
+			(justify left bottom)
+		)
+	)
+	(label "CinP"
+		(at 85.09 158.75 0)
 		(effects
 			(font
@@
 	(label "LMK13_plane"
 		(at 74.93 44.45 0)
-		(fields_autoplaced yes)
 		(effects
 			(font
@@
 	(label "ADC1_CLK-"
 		(at 106.68 55.88 180)
-		(fields_autoplaced yes)
 		(effects
 			(font
@@
 	(label "ADC0_CLK+"
 		(at 132.08 63.5 180)
-		(fields_autoplaced yes)
 		(effects
 			(font
@@
 	(label "LEuWire_CLKoutDIV_2"
 		(at 143.51 50.8 180)
-		(fields_autoplaced yes)
 		(effects
 			(font
@@
 	(label "LMK57_plane"
 		(at 64.77 54.61 0)
-		(fields_autoplaced yes)
 		(effects
 			(font
@@
 	(label "LMK13_plane"
 		(at 132.08 33.02 0)
-		(fields_autoplaced yes)
-		(effects
-			(font
-				(size 1.27 1.27)
-			)
-			(justify left bottom)
-		)
-	)
-	(label "aux_clk_n"
+		(effects
+			(font
+				(size 1.27 1.27)
+			)
+			(justify left bottom)
+		)
+	)
+	(label "aux_clk_N"
 		(at 172.72 152.4 180)
-		(fields_autoplaced yes)
 		(effects
 			(font
@@
 	(label "CLKinP"
 		(at 101.6 158.75 0)
-		(fields_autoplaced yes)
 		(effects
 			(font
@@
 	(label "LMK_CLKout3_P"
 		(at 143.51 81.28 180)
-		(fields_autoplaced yes)
 		(effects
 			(font
@@
 	(label "DATAuWire_CLKoutDIV_0"
 		(at 143.51 40.64 180)
-		(fields_autoplaced yes)
 		(effects
 			(font
@@
 	(label "CLKinN"
 		(at 143.51 99.06 180)
-		(fields_autoplaced yes)
 		(effects
 			(font
@@
 	(label "CLKinN"
 		(at 245.11 76.2 0)
-		(fields_autoplaced yes)
 		(effects
 			(font
@@
 	(label "CLKinP"
 		(at 143.51 96.52 180)
-		(fields_autoplaced yes)
 		(effects
 			(font
@@
 	(label "LMK2468_plane"
 		(at 129.54 25.4 0)
-		(fields_autoplaced yes)
 		(effects
 			(font
@@
 	(label "CLKuWire_CLKoutDIV_1"
 		(at 143.51 45.72 180)
-		(fields_autoplaced yes)
 		(effects
 			(font
@@
 	(label "LMK57_plane"
 		(at 245.11 30.48 0)
-		(fields_autoplaced yes)
-		(effects
-			(font
-				(size 1.27 1.27)
-			)
-			(justify left bottom)
-		)
-	)
-	(label "aux_clk_n"
+		(effects
+			(font
+				(size 1.27 1.27)
+			)
+			(justify left bottom)
+		)
+	)
+	(label "aux_clk_N"
 		(at 246.38 91.44 0)
-		(fields_autoplaced yes)
 		(effects
 			(font
@@
 	(label "LMK2468_plane"
 		(at 245.11 25.4 0)
-		(fields_autoplaced yes)
 		(effects
 			(font
@@
 	(label "LMK57_plane"
 		(at 245.11 33.02 0)
-		(fields_autoplaced yes)
 		(effects
 			(font
@@
 	(label "LMK13_plane"
 		(at 132.08 30.48 0)
-		(fields_autoplaced yes)
 		(effects
 			(font
@@
 	(label "DAC_CLKP"
 		(at 123.19 114.3 0)
-		(fields_autoplaced yes)
 		(effects
 			(font
@@
 	(label "ADC1_CLK+"
 		(at 106.68 58.42 180)
-		(fields_autoplaced yes)
 		(effects
 			(font
@@
 	(label "LMK_CLKout4_N"
 		(at 143.51 106.68 180)
-		(fields_autoplaced yes)
 		(effects
 			(font
@@
 	(label "LMK2468_plane"
 		(at 245.11 43.18 0)
-		(fields_autoplaced yes)
+		(effects
+			(font
+				(size 1.27 1.27)
+			)
+			(justify left bottom)
+		)
+	)
+	(label "CinN"
+		(at 85.09 151.13 0)
 		(effects
 			(font
@@
 		(shape input)
 		(at 91.44 60.96 0)
-		(fields_autoplaced yes)
 		(effects
 			(font
@@
 		(shape input)
 		(at 95.25 135.89 0)
-		(fields_autoplaced yes)
 		(effects
 			(font
@@
 		(shape input)
 		(at 109.22 111.76 180)
-		(fields_autoplaced yes)
 		(effects
 			(font
@@
 		(shape input)
 		(at 115.57 40.64 180)
-		(fields_autoplaced yes)
 		(effects
 			(font
@@
 		(shape input)
 		(at 121.92 78.74 180)
-		(fields_autoplaced yes)
 		(effects
 			(font
@@
 		(shape input)
 		(at 115.57 73.66 180)
-		(fields_autoplaced yes)
 		(effects
 			(font
@@
 		(shape input)
 		(at 30.48 44.45 180)
-		(fields_autoplaced yes)
-		(effects
-			(font
+		(effects
+			(font
