File: lmk01801.kicad_sch (KiCad schematic)
At the start: 41 parts, among them J1001 142-0701-201, J1002 U.FL-R-SMT(10), J1003 U.FL-R-SMT(10), J1004 142-0701-201, J1005 U.FL-R-SMT(10), T1001 TCM2-43X+, T1002 TCM2-43X+, U1001 TCP-2-33W+, U1002 LMK01801BISQE/NOPB

Commit message: fixed differential pair impedance and length matching. Also fixed DRC errors (trace spacing). These are only layout changes, the schematic remains unchanged.
Connections:
- net CinP: now reaches C1007.1, R1002.1, T1001.4
- net CinN: now reaches C1006.1, R1002.2, T1001.6
- net aux_clk_n renamed aux_clk_N
- net aux_clk_p renamed aux_clk_P
Changed lines of the file:
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@@
 		)
 	)
-	(label "aux_clk_p"
+	(label "aux_clk_P"
 		(at 246.38 93.98 0)
 		(effects
@@
 		)
 	)
-	(label "aux_clk_p"
+	(label "aux_clk_P"
 		(at 172.72 149.86 180)
 		(effects
@@
 		)
 	)
+	(label "CinP"
+		(at 85.09 158.75 0)
+		(effects
+			(font
+				(size 1.27 1.27)
+			)
+			(justify left bottom)
+		)
+	)
 	(label "LMK13_plane"
 		(at 74.93 44.45 0)
@@
 		)
 	)
-	(label "aux_clk_n"
+	(label "aux_clk_N"
 		(at 172.72 152.4 180)
 		(effects
@@
 		)
 	)
-	(label "aux_clk_n"
+	(label "aux_clk_N"
 		(at 246.38 91.44 0)
 		(effects
@@
 		(effects
 			(font
+				(size 1.27 1.27)
+			)
+			(justify left bottom)
+		)
+	)
+	(label "CinN"
+		(at 85.09 151.13 0)
+		(effects
+			(font
