File: se_diff.kicad_sch (KiCad schematic)
At the start: 12 parts

Commit message: fixed differential pair impedance and length matching. Also fixed DRC errors (trace spacing). These are only layout changes, the schematic remains unchanged.
Parts:
- renumbered C2301 to C301, C2302 to C302, C2303 to C303, C2304 to C304, L2301 to L301, R2301 to R301, R2302 to R302, R2303 to R303, R2304 to R304, R2305 to R305, R2306 to R306, XMER2301 to XMER301
Changed lines of the file:
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@@
 (kicad_sch
-	(version 20231120)
+	(version 20250114)
 	(generator "eeschema")
-	(generator_version "8.0")
+	(generator_version "9.0")
 	(paper "A4")
 	(junction
@@
 		(shape input)
 		(at 90.17 76.2 180)
-		(fields_autoplaced yes)
 		(effects
 			(font
@@
 		(shape input)
 		(at 231.14 83.82 0)
-		(fields_autoplaced yes)
 		(effects
 			(font
@@
 		(shape input)
 		(at 90.17 81.28 180)
-		(fields_autoplaced yes)
 		(effects
 			(font
@@
 		(shape input)
 		(at 231.14 91.44 0)
-		(fields_autoplaced yes)
 		(effects
 			(font
@@
 		(shape input)
 		(at 231.14 73.66 0)
-		(fields_autoplaced yes)
 		(effects
 			(font
@@
 		(on_board yes)
 		(dnp no)
-		(property "Reference" "R2306"
+		(property "Reference" "R306"
 			(at 227.33 90.17 90)
 			(effects
@@
 		(dnp no)
 		(fields_autoplaced yes)
-		(property "Reference" "L2301"
+		(property "Reference" "L301"
 			(at 218.44 78.7399 0)
 			(effects
@@
 		(dnp no)
 		(fields_autoplaced yes)
-		(property "Reference" "XMER2301"
+		(property "Reference" "XMER301"
 			(at 135.89 66.04 0)
 			(effects
@@
 		(on_board yes)
 		(dnp no)
-		(property "Reference" "C2302"
+		(property "Reference" "C302"
 			(at 93.98 88.9 90)
 			(effects
@@
 		(on_board yes)
 		(dnp no)
-		(property "Reference" "C2301"
+		(property "Reference" "C301"
 			(at 93.98 68.58 90)
 			(effects
@@
 		(dnp no)
 		(fields_autoplaced yes)
-		(property "Reference" "R2303"
+		(property "Reference" "R303"
 			(at 198.12 77.4699 0)
 			(effects
@@
 		(on_board yes)
 		(dnp no)
-		(property "Reference" "R2301"
+		(property "Reference" "R301"
 			(at 185.42 67.31 90)
 			(effects
@@
 		(on_board yes)
 		(dnp no)
-		(property "Reference" "R2302"
+		(property "Reference" "R302"
 			(at 185.42 90.17 90)
 			(effects
@@
 		(dnp no)
 		(fields_autoplaced yes)
-		(property "Reference" "C2304"
+		(property "Reference" "C304"
 			(at 210.82 77.4699 0)
 			(effects
@@
 		(on_board yes)
 		(dnp no)
-		(property "Reference" "C2303"
+		(property "Reference" "C303"
 			(at 182.88 99.0601 0)
 			(effects
@@
 		(dnp no)
 		(fields_autoplaced yes)
-		(property "Reference" "#PWR02301"
+		(property "Reference" "#PWR0301"
 			(at 179.07 107.95 0)
 			(effects
@@
 		(on_board yes)
 		(dnp no)
-		(property "Reference" "R2305"
+		(property "Reference" "R305"
 			(at 227.33 80.01 90)
 			(effects
@@
 		(on_board yes)
 		(dnp no)
-		(property "Reference" "R2304"
+		(property "Reference" "R304"
 			(at 204.47 97.79 90)
 			(effects
