File: thermo_bridge.kicad_sch (KiCad schematic)
At the start: 4 parts

Commit message: fixed differential pair impedance and length matching. Also fixed DRC errors (trace spacing). These are only layout changes, the schematic remains unchanged.
Parts:
- renumbered R3601 to R3301, R3602 to R3302, R3603 to R3303, R3604 to R3304
Changed lines of the file:
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@@
 (kicad_sch
-	(version 20231120)
+	(version 20250114)
 	(generator "eeschema")
-	(generator_version "8.0")
+	(generator_version "9.0")
 	(paper "A4")
 	(junction
@@
 		(shape input)
 		(at 78.74 87.63 180)
-		(fields_autoplaced yes)
 		(effects
 			(font
@@
 		(shape input)
 		(at 113.03 102.87 0)
-		(fields_autoplaced yes)
 		(effects
 			(font
@@
 		(shape input)
 		(at 113.03 77.47 0)
-		(fields_autoplaced yes)
 		(effects
 			(font
@@
 		(shape input)
 		(at 107.95 93.98 0)
-		(fields_autoplaced yes)
 		(effects
 			(font
@@
 		(on_board yes)
 		(dnp no)
-		(property "Reference" "R3602"
+		(property "Reference" "R3302"
 			(at 90.17 100.33 90)
 			(effects
@@
 		(on_board yes)
 		(dnp no)
-		(property "Reference" "R3601"
+		(property "Reference" "R3301"
 			(at 90.17 81.28 90)
 			(effects
@@
 		(dnp no)
 		(fields_autoplaced yes)
-		(property "Reference" "R3603"
+		(property "Reference" "R3303"
 			(at 97.79 81.28 90)
 			(effects
@@
 		(on_board yes)
 		(dnp no)
-		(property "Reference" "R3604"
+		(property "Reference" "R3304"
 			(at 97.79 100.33 90)
 			(effects
