File: zest.kicad_pcb (KiCad board)
At the start: 8 copper layers, 110 x 181.8 mm, 443 parts, among them J1001 142-0701-201, J1002 U.FL-R-SMT(10), J1003 U.FL-R-SMT(10), J1004 142-0701-201, J1005 U.FL-R-SMT(10), J1201 142-0701-201, J1202 142-0701-201, J1401 ASP-134604-01, J1402 ASP-134604-01, J1501 10029449-111RLF, J1502 PPPC072LJBN-RC, J1503 PPPC072LJBN-RC, J1901 961102-6404-AR, J201 142-0701-201, J202 142-0701-201, J203 142-0701-201, J204 142-0701-201, J701 142-0701-201, J702 142-0701-201, J703 142-0701-201, J704 142-0701-201, J801 20021121-00020C4LF, J802 20021121-00020C4LF, J901 U.FL-R-SMT(10), J902 U.FL-R-SMT(10), J903 U.FL-R-SMT(10), J904 U.FL-R-SMT(10), J905 U.FL-R-SMT(10), J906 U.FL-R-SMT(10), Q1501 FDN335N, Q1502 FDN335N, T1001 TCM2-43X+, T1002 TCM2-43X+, U1001 TCP-2-33W+, U1002 LMK01801BISQE/NOPB, U1101 AD7794BRUZ, U1201 AD9781BCPZ, U1301 AMC7823IRTAT, U1601 LT6233CS6#TRMPBF, U1701 SN74LVC8T245PWR, U1702 SN74LVC8T245PWR, U1703 SN74LVC8T245PWR, U1704 SN74AVC4T245PWR, U1705 SN74AVC4T245PWR, U1801 ADL5501AKSZ-R7, U1901 AT24C64D-SSHM-T, U2001 KX023-1025-FR, U201 AD9653BCPZ-125, U2701 TPS62110RSAR, U2801 LTC6655CHLS8-2.5#PBF, U2901 TPS62110RSAR, U3001 LT6233CS6#TRMPBF, U3002 PBSS4230T,215, U3101 LT1763IDE-3.3#PBF, U3201 LT1763IDE-1.8#PBF, U701 AD9653BCPZ-125, U901 BAT54W-7-F, U902 ZXCT1009QFTA, U903 LT6233CS6#TRMPBF

Commit message: fixed differential pair impedance and length matching. Also fixed DRC errors (trace spacing). These are only layout changes, the schematic remains unchanged.
Parts:
- removed TP33, TP34: TestPoint, 001_download:TestPoint_Pad_D0.6mm
- moved C1004 258.1 mm to (47.0, 33.6)
- moved R3501 257.8 mm to (95.6, 80.9)
- moved R3502 257.8 mm to (91.8, 80.9)
- moved R3503 257.8 mm to (95.6, 79.0)
- moved R3504 257.8 mm to (91.8, 79.0)
- moved R2406 253.7 mm to (47.6, 160.9), turned to 0 degrees
- moved R2405 253.4 mm to (47.6, 159.4), turned to 0 degrees
- moved R306 253.0 mm to (47.6, 99.8), turned to 0 degrees
- moved R305 252.8 mm to (47.6, 98.3), turned to 0 degrees
- moved R901 252.6 mm to (108.8, 139.4), turned to -90 degrees
- moved C2705 252.6 mm to (77.9, 60.3)
- moved C2404 251.5 mm to (45.3, 160.2), turned to -90 degrees
- moved C304 250.9 mm to (45.4, 99.1), turned to -90 degrees
- moved J904 248.4 mm to (81.8, 63.6), turned to -90 degrees
- moved C710 246.9 mm to (42.6, 105.1), turned to -90 degrees
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Connections:
- net /lmk01801/aux_clk_n renamed /lmk01801/aux_clk_N
- net /lmk01801/aux_clk_p renamed /lmk01801/aux_clk_P
- net Net-(C1006-Pad1) renamed /lmk01801/CinN
- net Net-(C1007-Pad1) renamed /lmk01801/CinP
- net Net-(U1201-CLKN) renamed /ad9781/D_CLKN
- net Net-(U1201-CLKP) renamed /ad9781/D_CLKP
- net Net-(U201-CLK+) renamed /ADC0/A0_CLK+
- net Net-(U201-CLK-) renamed /ADC0/A0_CLK-
- net Net-(U701-CLK+) renamed /ADC1/A1_CLK+
- net Net-(U701-CLK-) renamed /ADC1/A1_CLK-
Routing:
- net GND: track 985.5 -> 589.9 mm, vias 527 -> 562
- net /VDD3P3V: track 627.5 -> 394.9 mm, vias 43 -> 40
- net /VSS3P3V: track 146.1 -> 19.7 mm, vias 19 -> 20
- net /P2_3P3V: track 6.66 -> 121.2 mm, vias 7 -> 4
- net /PowerSupply/DC3P7V: track 104.2 -> 77.1 mm, vias 8 -> 2
- net Net-(C604-Pad1): track 32.0 -> 5.90 mm
- net Net-(C2304-Pad1): track 31.2 -> 5.90 mm
- net Net-(C604-Pad2): track 31.1 -> 5.90 mm
- net Net-(C2404-Pad2): track 30.9 -> 5.85 mm
- net Net-(C304-Pad2): track 30.5 -> 5.85 mm
- net Net-(C2404-Pad1): track 30.4 -> 5.90 mm
- net Net-(C2304-Pad2): track 30.3 -> 5.85 mm
- net Net-(C304-Pad1): track 28.9 -> 5.90 mm
- net (no net): track 22.0 -> 0.00 mm
- net /ADC0/se2diff_0/CM: track 77.1 -> 98.4 mm
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- added copper zone on F.Cu, net /P2_3P3V
- added copper zone on F.Cu, net /PowerSupply/DC2P2V
- added copper zone on F.Cu, net /PowerSupply/DC3P7V
- added copper zone on F.Cu, net /VDD1P8V
- added copper zone on F.Cu, net /VSS1P8V
- added copper zone on F.Cu, net /VSS3P3V
- added copper zone on F.Cu, net GND
- added copper zone on F.Cu, net Net-(U2701-VINA)
- added copper zone on F.Cu, net Net-(U2901-VINA)
- added copper zone on F.Cu, net Net-(U3101-IN)
- added copper zone on F.Cu, net Net-(U3201-IN)
- removed copper zone on In6.Cu, net /P2_3P3V
Other:
- board text added: "0"
- board text added: "0 mm"
- board text added: "0.01 mm"
- board text added: "0.02"
- board text added: "0.035 mm"
- board text added: "0.043 mm"
- board text added: "0.165 mm"
- board text added: "0.2 mm"
- board text added: "1"
- board text added: "2"
- board text added: "3"
- board text added: "3.3"
- board text added: "4"
- board text added: "4.5"
- board text added: "5"
- board text added: "6"
- board text added: "8"
- board text added: "B.Cu"
- board text added: "B.Mask"
- board text added: "B.Paste"
- board text added: "B.Silkscreen"
- board text added: "Bottom Silk Screen"
- board text added: "Bottom Solder Mask"
- board text added: "Bottom Solder Paste"
- board text added: "Color"
- board text added: "Dielectric 1"
- board text added: "Dielectric 2"
- board text added: "Dielectric 3"
- board text added: "Dielectric 4"
- board text added: "Dielectric 5"
- board text added: "Dielectric 6"
- board text added: "Dielectric 7"
- board text added: "Epsilon R"
- board text added: "F.Cu"
- board text added: "F.Mask"
- board text added: "F.Paste"
- board text added: "F.Silkscreen"
- board text added: "FR4"
- board text added: "In1.Cu"
- board text added: "In2.Cu"
- board text added: "In3.Cu"
- board text added: "In4.Cu"
- board text added: "In5.Cu"
- board text added: "In6.Cu"
- board text added: "Layer Name"
- board text added: "Loss Tangent"
- board text added: "Material"
- board text added: "Not specified"
- board text added: "Thickness (mm)"
- board text added: "Top Silk Screen"
- board text added: "Top Solder Mask"
- board text added: "Top Solder Paste"
- board text added: "Type"
- board text added: "ZEST"
- board text added: "copper"
- board text added: "core"
- board text added: "prepreg"
- board text added: "ver 1.3 G. H., M. G., S. W."
- board text added: "ver 1.3 G.H., M.G., S.W."
- board text removed: "Zest ver 1.2 By G. H"
